Commit message: big update

File: src/my_robot_world/urdf/conveyorbelt_product.urdf.xacro (robot description, xacro)
@@ -2,5 +2,5 @@
 <robot name="conveyor_belt_product">
 <!-- conveyor belt is just a long flat box for objects to slide on it -->
- world link
+<!-- world link-->
 <link name="world"/>
 <!-- base_link and its fixed joint -->

File: src/my_robot_world/urdf/myRobot.urdf.xacro (robot description, xacro)
@@ -23,5 +23,5 @@
     <parent link="table_link" />
     <child link = "base_link" />
-    <origin xyz="0.0 0.0 0.7" rpy="0.0 0.0 0.0" />
+    <origin xyz="0.0 0.0 0.701" rpy="0.0 0.0 0.0" />
   </joint>
 </robot>

File: src/my_robot_world/urdf/table.urdf.xacro (robot description, xacro)
@@ -15,4 +15,10 @@
       </geometry>
     </visual>
+    <collision>
+	    <origin rpy="0.0 0 0" xyz="0 0 0.35"/>
+	    <geometry>
+	      <cylinder radius="0.3" length="0.7" />
+	    </geometry>
+  	</collision>
     <inertial>
       <origin xyz="0 0 0.35" rpy="0 0 0"/>
